Commit message: model is ready for the gym

File: urdf/delta_robot_pybullet.urdf (robot description, URDF)
Before this commit: robot delta-robot-RUU, 20 links, 19 joints
Links:
- link world: mass 1e-05 -> None; geometry 

File: urdf/delta_robot_pybullet.urdf.xacro (robot description, xacro)
@@ -145,10 +145,5 @@
                          axis="z"
                          mat="heart_pink" />
-  <xacro:cylinder_link name="world"
-                       M="1e-5"
-                       R="1e-5"
-                       h="1e-5"
-                       axis="x"
-                       mat="base_color" />
+  <link name="world"/>
   <!-- connect the base to the world -->
   <joint name="fixed" type="fixed">
